Commit message: in RoboterArm-xacro Kamera_node hinzugefügt

File: src/robotik_description/urdf/ur5e.urdf.xacro (robot description, xacro)
@@ -16,3 +16,31 @@
     <origin xyz="0 0 0.2" rpy="0 0 0"/>
   </xacro:ur_robot>
+    <!-- Kamera am Greifer / tool0 -->
+  <link name="camera_link">
+    <visual>
+      <geometry>
+        <box size="0.05 0.03 0.03"/>
+      </geometry>
+      <material name="camera_black">
+        <color rgba="0.0 0.0 0.0 255.0"/>
+      </material>
+    </visual>
+    <collision>
+      <geometry>
+        <box size="0.05 0.03 0.03"/>
+      </geometry>
+    </collision>
+    <inertial>
+      <mass value="0.05"/>
+      <origin xyz="0 0 0"/>
+      <inertia ixx="0.00001" ixy="0.0" ixz="0.0"
+               iyy="0.00001" iyz="0.0"
+               izz="0.00001"/>
+    </inertial>
+  </link>
+  <joint name="camera_joint" type="fixed">
+    <parent link="tool0"/>
+    <child link="camera_link"/>
+    <origin xyz="-0.063 0 -0.03" rpy="0 0 0"/>
+  </joint>
 </robot>

Commit message: OpenCV hinzugefügt

File: src/robotik_description/urdf/ur5e.urdf.xacro (robot description, xacro)
@@ -16,51 +16,44 @@
     <origin xyz="0 0 0.2" rpy="0 0 0"/>
   </xacro:ur_robot>
-    <!-- Kamera am Greifer / tool0 -->
-  <link name="camera_link">
-    <visual>
-      <geometry>
-        <box size="0.05 0.03 0.03"/>
-      </geometry>
-      <material name="camera_black">
-        <color rgba="0.0 0.0 0.0 1.0"/>
-      </material>
-    </visual>
-    <collision>
-      <geometry>
-        <box size="0.05 0.03 0.03"/>
-      </geometry>
-    </collision>
-    <inertial>
-      <mass value="0.05"/>
-      <origin xyz="0 0 0"/>
-      <inertia ixx="0.00001" ixy="0.0" ixz="0.0"
-               iyy="0.00001" iyz="0.0"
-               izz="0.00001"/>
-    </inertial>
-  </link>
-  <joint name="camera_joint" type="fixed">
-    <parent link="tool0"/>
-    <child link="camera_link"/>
-    <origin xyz="-0.063 0 -0.03" rpy="0 0 0"/>
-  </joint>
-    <gazebo reference="camera_link">
-    <sensor name="gripper_depth_camera" type="rgbd_camera">
-      <pose>0 0 0 0 0 0</pose>
-      <always_on>1</always_on>
-      <update_rate>30</update_rate>
-      <topic>gripper_depth_camera</topic>
-      <camera>
-        <horizontal_fov>1.047</horizontal_fov>
-        <image>
-          <width>640</width>
-          <height>480</height>
-          <format>R8G8B8</format>
-        </image>
-        <clip>
-          <near>0.05</near>
-          <far>5.0</far>
-        </clip>
-      </camera>
-    </sensor>
+     <ros2_control name="UR5eSystem" type="system">
+    <hardware>
+      <plugin>gz_ros2_control/GazeboSimSystem</plugin>
+    </hardware>
+    <joint name="shoulder_pan_joint">
+      <command_interface name="position"/>
+      <state_interface name="position"/>
+      <state_interface name="velocity"/>
+    </joint>
+    <joint name="shoulder_lift_joint">
+      <command_interface name="position"/>
+      <state_interface name="position"/>
+      <state_interface name="velocity"/>
+    </joint>
+    <joint name="elbow_joint">
+      <command_interface name="position"/>
+      <state_interface name="position"/>
+      <state_interface name="velocity"/>
+    </joint>
+    <joint name="wrist_1_joint">
+      <command_interface name="position"/>
+      <state_interface name="position"/>
+      <state_interface name="velocity"/>
+    </joint>
+    <joint name="wrist_2_joint">
+      <command_interface name="position"/>
+      <state_interface name="position"/>
+      <state_interface name="velocity"/>
+    </joint>
+    <joint name="wrist_3_joint">
+      <command_interface name="position"/>
+      <state_interface name="position"/>
+      <state_interface name="velocity"/>
+    </joint>
+  </ros2_control>
+  <gazebo>
+    <plugin filename="gz_ros2_control-system"
+            name="gz_ros2_control::GazeboSimROS2ControlPlugin">
+      <parameters>$(find robotik_control)/config/ur5e_controllers.yaml</parameters>
+    </plugin>
   </gazebo>
 </robot>

Commit message: Stable vision and UR5e RViz state before ros2_control

File: src/robotik_description/urdf/ur5e.urdf.xacro (robot description, xacro)
@@ -16,44 +16,3 @@
     <origin xyz="0 0 0.2" rpy="0 0 0"/>
   </xacro:ur_robot>
-     <ros2_control name="UR5eSystem" type="system">
-    <hardware>
-      <plugin>gz_ros2_control/GazeboSimSystem</plugin>
-    </hardware>
-    <joint name="shoulder_pan_joint">
-      <command_interface name="position"/>
-      <state_interface name="position"/>
-      <state_interface name="velocity"/>
-    </joint>
-    <joint name="shoulder_lift_joint">
-      <command_interface name="position"/>
-      <state_interface name="position"/>
-      <state_interface name="velocity"/>
-    </joint>
-    <joint name="elbow_joint">
-      <command_interface name="position"/>
-      <state_interface name="position"/>
-      <state_interface name="velocity"/>
-    </joint>
-    <joint name="wrist_1_joint">
-      <command_interface name="position"/>
-      <state_interface name="position"/>
-      <state_interface name="velocity"/>
-    </joint>
-    <joint name="wrist_2_joint">
-      <command_interface name="position"/>
-      <state_interface name="position"/>
-      <state_interface name="velocity"/>
-    </joint>
-    <joint name="wrist_3_joint">
-      <command_interface name="position"/>
-      <state_interface name="position"/>
-      <state_interface name="velocity"/>
-    </joint>
-  </ros2_control>
-  <gazebo>
-    <plugin filename="gz_ros2_control-system"
-            name="gz_ros2_control::GazeboSimROS2ControlPlugin">
-      <parameters>$(find robotik_control)/config/ur5e_controllers.yaml</parameters>
-    </plugin>
-  </gazebo>
 </robot>

Commit message: alle  was  gemacht ist

File: src/robotik_description/urdf/ur5e.urdf.xacro (robot description, xacro)
@@ -16,3 +16,44 @@
     <origin xyz="0 0 0.2" rpy="0 0 0"/>
   </xacro:ur_robot>
+    <ros2_control name="UR5eSystem" type="system">
+    <hardware>
+      <plugin>gz_ros2_control/GazeboSimSystem</plugin>
+    </hardware>
+    <joint name="shoulder_pan_joint">
+      <command_interface name="position"/>
+      <state_interface name="position"/>
+      <state_interface name="velocity"/>
+    </joint>
+    <joint name="shoulder_lift_joint">
+      <command_interface name="position"/>
+      <state_interface name="position"/>
+      <state_interface name="velocity"/>
+    </joint>
+    <joint name="elbow_joint">
+      <command_interface name="position"/>
+      <state_interface name="position"/>
+      <state_interface name="velocity"/>
+    </joint>
+    <joint name="wrist_1_joint">
+      <command_interface name="position"/>
+      <state_interface name="position"/>
+      <state_interface name="velocity"/>
+    </joint>
+    <joint name="wrist_2_joint">
+      <command_interface name="position"/>
+      <state_interface name="position"/>
+      <state_interface name="velocity"/>
+    </joint>
+    <joint name="wrist_3_joint">
+      <command_interface name="position"/>
+      <state_interface name="position"/>
+      <state_interface name="velocity"/>
+    </joint>
+  </ros2_control>
+  <gazebo>
+    <plugin filename="libgz_ros2_control-system.so"
+            name="gz_ros2_control::GazeboSimROS2ControlPlugin">
+      <parameters>$(find robotik_control)/config/ur5e_controllers.yaml</parameters>
+    </plugin>
+  </gazebo>
 </robot>

Commit message: it hurts when ip

File: src/robotik_description/urdf/ur5e.urdf.xacro (robot description, xacro)
@@ -3,4 +3,5 @@
   <link name="world"/>
   <xacro:include filename="$(find ur_description)/urdf/ur_macro.xacro"/>
+  <xacro:include filename="$(find robotik_description)/urdf/simple_gripper.urdf.xacro"/>
   <xacro:ur_robot
     name="ur5e"
@@ -50,5 +51,16 @@
       <state_interface name="velocity"/>
     </joint>
+    <joint name="left_finger_joint">
+      <command_interface name="position"/>
+      <state_interface name="position"/>
+      <state_interface name="velocity"/>
+    </joint>
+    <joint name="right_finger_joint">
+      <command_interface name="position"/>
+      <state_interface name="position"/>
+      <state_interface name="velocity"/>
+    </joint>
   </ros2_control>
+  <xacro:simple_gripper parent_link="tool0"/>
   <gazebo>
     <plugin filename="libgz_ros2_control-system.so"
